Commit message: Manual point streaming & debug messages

File: motoman_sda10f_support/urdf/common_torso_macro.xacro (robot description, xacro)
@@ -39,5 +39,5 @@
 			</collision>
 		</link>
-		<link name="${prefix}link_b2">
+		<!--link name="${prefix}link_b2">
 			<visual>
 				<origin rpy="0 0 0" xyz="0 0 0"/>
@@ -56,5 +56,5 @@
 				<material name="yellow"/>
 			</collision>
-		</link>
+		</link-->
 		<!-- joint list -->
 		<joint name="${prefix}joint_b1" type="revolute">
@@ -65,12 +65,12 @@
 			<limit lower="-2.9570" upper="2.9570" effort="100" velocity="2.26" />
 		</joint>
-		<joint name="${prefix}joint_b2" type="revolute">
+		<!--joint name="${prefix}joint_b2" type="fixed">
 			<parent link="${prefix}base_link"/>
 			<child link="${prefix}link_b2"/>
 			<origin xyz="0.09257 0 0.8835" rpy="0 0 0"/>
 			<axis xyz="0 0 1" />
-			<limit lower="-2.9570" upper="2.9570" effort="100" velocity="2.26" />
-			<mimic joint="${prefix}joint_b1" multiplier="1" offset="0"/>
-		</joint>
+			<limit lower="-2.9570" upper="2.9570" effort="100" velocity="2.26" /-->
+			<!--mimic joint="${prefix}joint_b1" multiplier="1" offset="0"/-->
+		<!--/joint-->
 		<!-- end of joint list -->
 	</xacro:macro>

File: motoman_sda10f_support/urdf/sda10f.xacro (robot description, xacro)
@@ -2,4 +2,17 @@
 <robot name="motoman_sda10f" xmlns:xacro="http://ros.org/wiki/xacro">
 	<xacro:include filename="$(find motoman_sda10f_support)/urdf/sda10f_macro.xacro" />
+    <xacro:include filename="$(find robot_setup_sda10f)/urdf/table.urdf.xacro" />
+    <xacro:include filename="$(find robot_setup_sda10f)/urdf/cover.urdf.xacro" />
+    <xacro:include filename="$(find wsg_50_simulation)/urdf/wsg_50.urdf.xacro" />
 	<xacro:motoman_sda10f prefix=""/>
+	<!-- ==============add table robot arm=================== -->
+    <xacro:table_model prefix="" parent="base_link">
+        <origin xyz="0.0 0.0 -0.16" rpy="${pi} 0 0" />
+    </xacro:table_model>
+    <xacro:cover_model prefix="" parent="arm_left_link_tool0">
+        <origin xyz="0.0 0.0 -0.04" rpy="${pi} 0 ${pi/2 + 0.29}" />
+    </xacro:cover_model>
+    <xacro:wsg_50_xacro name="wsg_50_gripper" parent="arm_left_link_tool0">
+        <origin xyz="0.0 0.0 -0.177" rpy="0 0 ${pi + 0.29}" />
+    </xacro:wsg_50_xacro>
 </robot>

File: motoman_sda10f_support/urdf/sda10f_macro.xacro (robot description, xacro)
@@ -17,3 +17,11 @@
           <xacro:motoman_sda10f prefix=""/>
      </xacro:macro>
+    		<!-- link list -->
+    <link name="base_link"> </link>
+    <joint name="torso_base_joint" type="fixed">
+        <parent link="base_link"/>
+        <child link="torso_base_link"/>
+        <origin xyz="0.0 0 0.0" rpy="0 0 0"/>
+        <axis xyz="0 0 1" />
+    </joint>
 </robot>
