Commit message: added pi parameter

File: motoman_sda10f_support/urdf/arm_macro.xacro (robot description, xacro)
@@ -118,5 +118,5 @@
 			<parent link="${parent}"/>
 			<child link="${prefix}link_1_s"/>
-			<origin xyz="0.09996 ${reflect*0.0275} 0.32214" rpy="1.57 0 ${(reflect-1)*1.57}"/>
+			<origin xyz="0.09996 ${reflect*0.0275} 0.32214" rpy="${pi/2} 0 ${(reflect-1)*pi/2}"/>
 			<axis xyz="0 0 ${-reflect}" />
 			<limit lower="-3.13" upper="3.13" effort="0" velocity="2.95" />
@@ -125,5 +125,5 @@
 			<parent link="${prefix}link_1_s"/>
 			<child link="${prefix}link_2_l"/>
-			<origin xyz="0 0.0577 -0.2255" rpy="-1.57 0 0"/>
+			<origin xyz="0 0.0577 -0.2255" rpy="-${pi/2} 0 0"/>
 			<axis xyz="0 0 ${-reflect}" />
 			<limit lower="-1.90" upper="1.90" effort="0" velocity="2.95" />
@@ -132,5 +132,5 @@
 			<parent link="${prefix}link_2_l"/>
 			<child link="${prefix}link_3_e"/>
-			<origin xyz="0 0.1690 -0.0454" rpy="1.57 0 0"/>
+			<origin xyz="0 0.1690 -0.0454" rpy="${pi/2} 0 0"/>
 			<axis xyz="0 0 ${-reflect}" />
 			<limit lower="-2.95" upper="2.95" effort="0" velocity="2.95" />
@@ -139,5 +139,5 @@
 			<parent link="${prefix}link_3_e"/>
 			<child link="${prefix}link_4_u"/>
-			<origin xyz="0 -0.0085 -0.181" rpy="-1.57 0 0"/>
+			<origin xyz="0 -0.0085 -0.181" rpy="-${pi/2} 0 0"/>
 			<axis xyz="0 0 ${reflect}" />
 			<limit lower="-2.36" upper="2.36" effort="0" velocity="2.95" />
@@ -146,5 +146,5 @@
 			<parent link="${prefix}link_4_u"/>
 			<child link="${prefix}link_5_r"/>
-			<origin xyz="0 0.1936 0.0155" rpy="1.57 0 0"/>
+			<origin xyz="0 0.1936 0.0155" rpy="${pi/2} 0 0"/>
 			<axis xyz="0 0 ${reflect}" />
 			<limit lower="-3.13" upper="3.13" effort="0" velocity="3.48" />
@@ -153,5 +153,5 @@
 			<parent link="${prefix}link_5_r"/>
 			<child link="${prefix}link_6_b"/>
-			<origin xyz="0 0.0080 -0.155" rpy="-1.57 0 0"/>
+			<origin xyz="0 0.0080 -0.155" rpy="-${pi/2} 0 0"/>
 			<axis xyz="0 0 ${reflect}" />
 			<limit lower="-1.90" upper="1.90" effort="0" velocity="3.48" />
@@ -160,10 +160,10 @@
 			<parent link="${prefix}link_6_b"/>
 			<child link="${prefix}link_7_t"/>
-			<origin xyz="0 0.168 -0.015" rpy="1.57 0 0"/>
+			<origin xyz="0 0.168 -0.015" rpy="${pi/2} 0 0"/>
 			<axis xyz="0 0 ${-reflect}" />
 			<limit lower="-3.13" upper="3.13" effort="0" velocity="6.97" />
 		</joint>
     <joint name="${prefix}joint_tool0" type="fixed" >
-      <origin xyz="0 0 0.0" rpy="0 0 -3.13"/>
+      <origin xyz="0 0 0.0" rpy="0 0 -${pi}"/>
       <parent link="${prefix}link_7_t" />
       <child link="${prefix}link_tool0" />

File: motoman_sda10f_support/urdf/sda10f.xacro (robot description, xacro)
@@ -2,17 +2,4 @@
 <robot name="motoman_sda10f" xmlns:xacro="http://ros.org/wiki/xacro">
 	<xacro:include filename="$(find motoman_sda10f_support)/urdf/sda10f_macro.xacro" />
-    <xacro:include filename="$(find robot_setup_sda10f)/urdf/table.urdf.xacro" />
-    <xacro:include filename="$(find robot_setup_sda10f)/urdf/cover.urdf.xacro" />
-    <xacro:include filename="$(find wsg_50_simulation)/urdf/wsg_50.urdf.xacro" />
-	<xacro:motoman_sda10f prefix=""/>
-	<!-- ==============add table robot arm=================== -->
-    <xacro:table_model prefix="" parent="base_link">
-        <origin xyz="0.0 0.0 -0.16" rpy="${pi} 0 0" />
-    </xacro:table_model>
-    <xacro:cover_model prefix="" parent="arm_left_link_tool0">
-        <origin xyz="0.0 0.0 -0.04" rpy="${pi} 0 ${pi/2 + 0.29}" />
-    </xacro:cover_model>
-    <xacro:wsg_50_xacro name="wsg_50_gripper" parent="arm_left_link_tool0">
-        <origin xyz="0.0 0.0 -0.177" rpy="0 0 ${pi + 0.29}" />
-    </xacro:wsg_50_xacro>
+    <xacro:motoman_sda10f prefix=""/>
 </robot>

File: motoman_sda10f_support/urdf/sda10f_macro.xacro (robot description, xacro)
@@ -3,11 +3,17 @@
      <xacro:include filename="$(find motoman_sda10f_support)/urdf/common_torso_macro.xacro" />
      <xacro:include filename="$(find motoman_sda10f_support)/urdf/arm_macro.xacro" />
-     <xacro:macro name="motoman_sda10f" params="prefix">
+     <xacro:property name="pi" value="3.1415926535898" />
+     <xacro:macro name="motoman_sda10f" params="prefix parent *origin">
+        <joint name="torso_base_joint" type="fixed">
+            <parent link="${parent}"/>
+            <child link="${prefix}torso_base_link"/>
+            <xacro:insert_block name="origin" />
+        </joint>
         <xacro:torso name="${prefix}torso" prefix="${prefix}torso_"/>
         <xacro:motoman_arm name="${prefix}arm_left" prefix="${prefix}arm_left_" parent="${prefix}torso_link_b1" reflect="1">
-            <origin xyz="0.09996 0.0275 0.32214" rpy="1.57 0 0" />
+            <origin xyz="0.09996 0.0275 0.32214" rpy="${pi/2} 0 0" />
         </xacro:motoman_arm>
         <xacro:motoman_arm name="${prefix}arm_right" prefix="${prefix}arm_right_" parent="${prefix}torso_link_b1" reflect="-1">
-            <origin xyz="0.09996 -0.0275 0.32214" rpy="1.57 0 0" />
+            <origin xyz="0.09996 -0.0275 0.32214" rpy="${pi/2} 0 0" />
         </xacro:motoman_arm>
      </xacro:macro>
@@ -17,5 +23,5 @@
           <xacro:motoman_sda10f prefix=""/>
      </xacro:macro>
-    		<!-- link list -->
+     <!-- link list -->
     <link name="base_link"> </link>
     <joint name="torso_base_joint" type="fixed">
